File: Configurable_RC_Filter.sch (EAGLE design)
At the start: 39 parts, among them SW1 DIP-06, SW2 DIP-06, SW3 DIP-06, SW4 DIP-06

Commit message: Change cap to NS package.
Parts:
- C12, C6: value 1mF -> 1000UF-RADIAL-5MM-25V-20%-NO-SILK; device SparkFun-Capacitors:1000UF-RADIAL-5MM-25V-20% -> SparkFun-Capacitors:1000UF-RADIAL-5MM-25V-20%-NO-SILK
Changed lines of the file:
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@@
 <part name="C4" library="SparkFun-Capacitors" deviceset="1.0UF" device="-0603-16V-10%" value="1.0uF"/>
 <part name="C5" library="SparkFun-Capacitors" deviceset="10UF" device="-0603-6.3V-20%" value="10uF"/>
-<part name="C6" library="SparkFun-Capacitors" deviceset="1000UF" device="-RADIAL-5MM-25V-20%" value="1mF"/>
+<part name="C6" library="SparkFun-Capacitors" deviceset="1000UF" device="-RADIAL-5MM-25V-20%-NO-SILK" value="1000UF-RADIAL-5MM-25V-20%-NO-SILK"/>
 <part name="GND1" library="SparkFun-PowerSymbols" deviceset="GND" device=""/>
 <part name="SUPPLY1" library="SparkFun-PowerSymbols" deviceset="VDDA" device=""/>
@@
 <part name="C10" library="SparkFun-Capacitors" deviceset="1.0UF" device="-0603-16V-10%" value="1.0uF"/>
 <part name="C11" library="SparkFun-Capacitors" deviceset="10UF" device="-0603-6.3V-20%" value="10uF"/>
-<part name="C12" library="SparkFun-Capacitors" deviceset="1000UF" device="-RADIAL-5MM-25V-20%" value="1mF"/>
+<part name="C12" library="SparkFun-Capacitors" deviceset="1000UF" device="-RADIAL-5MM-25V-20%-NO-SILK" value="1000UF-RADIAL-5MM-25V-20%-NO-SILK"/>
 <part name="SW4" library="SparkFun-Switches" deviceset="DIP-06" device=""/>
 <part name="R7" library="SparkFun-Resistors" deviceset="10MOHM" device="-0603-1/10W-5%" value="10M"/>
@@
 <instance part="C6" gate="G$1" x="106.68" y="101.6" smashed="yes">
 <attribute name="NAME" x="107.696" y="102.235" size="1.778" layer="95" font="vector"/>
-<attribute name="VALUE" x="107.696" y="97.409" size="1.778" layer="96" font="vector"/>
 </instance>
 <instance part="GND1" gate="1" x="93.98" y="88.9" smashed="yes">
@@
 <instance part="C12" gate="G$1" x="172.72" y="144.78" smashed="yes" rot="R90">
 <attribute name="NAME" x="170.815" y="141.224" size="1.778" layer="95" font="vector" rot="R270"/>
-<attribute name="VALUE" x="176.149" y="141.224" size="1.778" layer="96" font="vector" rot="R270"/>
 </instance>
 <instance part="SW4" gate="G$1" x="205.74" y="134.62" smashed="yes" rot="R180">
