File: Production/Configurable_RC_Filter-Panel.brd (EAGLE design)
At the start: 48.3 x 40.6 mm, 76 parts, among them SW1 DIP-06, SW2 DIP-06, SW3 DIP-06, SW4 DIP-06

Commit message: Add panel
Parts:
- removed FRAME1: FRAME-LETTER, SparkFun-Aesthetics:CREATIVE_COMMONS
- added C100, C106, C114, C120, C16, C22, C30, C36, C44, C50, C58, C64, C72, C78, C86, C92: 100pF, SparkFun-Capacitors:0603
- added C101, C107, C115, C121, C17, C23, C31, C37, C45, C51, C59, C65, C73, C79, C87, C93: 10nF, SparkFun-Capacitors:0603
- added C102, C108, C116, C122, C18, C24, C32, C38, C46, C52, C60, C66, C74, C80, C88, C94: 1.0uF, SparkFun-Capacitors:0603
- added C103, C109, C117, C123, C19, C25, C33, C39, C47, C53, C61, C67, C75, C81, C89, C95: 10uF, SparkFun-Capacitors:0603
- added C104, C110, C118, C124, C20, C26, C34, C40, C48, C54, C62, C68, C76, C82, C90, C96: 1000UF-RADIAL-5MM-25V-20%-NO-SILK, SparkFun-Capacitors:CPOL-RADIAL-5MM-10MM-NS
- added C105, C113, C119, C15, C21, C29, C35, C43, C49, C57, C63, C71, C77, C85, C91, C99: 1.0pF, SparkFun-Capacitors:0603
- added C111, C112, C125, C126, C27, C28, C41, C42, C55, C56, C69, C70, C83, C84, C97, C98: (no value), SparkFun-Capacitors:0603
- added E$1, E$2: (no value), SparkFun-Aesthetics:FIDUCIAL-1X2
- added E$3: (no value), SparkFun-Retired:FIDUCIAL-1.5X3
- added FD10, FD11, FD12, FD13, FD14, FD15, FD16, FD17, FD18, FD19, FD20, FD21, FD22, FD23, FD24, FD25, FD26, FD27, FD28, FD29, FD30, FD31, FD32, FD33, FD34, FD35, FD36, FD5, FD6, FD7, FD8, FD9: FIDUCIAL1X2, SparkFun-Aesthetics:FIDUCIAL-1X2
- added J2, J3, J4, J5, J6, J7, J8, J9: (no value), SparkFun-Connectors:1X04_NO_SILK
- added LOGO2, LOGO3, LOGO4, LOGO5, LOGO6, LOGO7, LOGO8, LOGO9: OSHW-LOGOS, SparkFun-Aesthetics:OSHW-LOGO-S
- added R100, R106, R114, R120, R16, R22, R30, R36, R44, R50, R58, R64, R72, R78, R86, R92: 100k, SparkFun-Resistors:0603
- added R101, R107, R115, R121, R17, R23, R31, R37, R45, R51, R59, R65, R73, R79, R87, R93: 1k, SparkFun-Resistors:0603
- added R102, R108, R116, R122, R18, R24, R32, R38, R46, R52, R60, R66, R74, R80, R88, R94: 1, SparkFun-Resistors:0603
- added R103, R109, R117, R123, R19, R25, R33, R39, R47, R53, R61, R67, R75, R81, R89, R95: 10, SparkFun-Resistors:0603
- added R104, R110, R118, R124, R20, R26, R34, R40, R48, R54, R62, R68, R76, R82, R90, R96: (no value), SparkFun-Resistors:AXIAL-0.3
- added R105, R113, R119, R15, R21, R29, R35, R43, R49, R57, R63, R71, R77, R85, R91, R99: 10M, SparkFun-Resistors:0603
- added R111, R112, R125, R126, R27, R28, R41, R42, R55, R56, R69, R70, R83, R84, R97, R98: (no value), SparkFun-Resistors:0603
- added SW10, SW11, SW12, SW13, SW14, SW15, SW16, SW17, SW18, SW19, SW20, SW21, SW22, SW23, SW24, SW25, SW26, SW27, SW28, SW29, SW30, SW31, SW32, SW33, SW34, SW35, SW36, SW5, SW6, SW7, SW8, SW9: DIP-06, SparkFun-Switches:DIPSWITCH-06-SMD
- added U$100, U$137, U$174, U$211, U$248, U$285, U$322, U$63: (no value), buzzard_labels (11):C20
- added U$101, U$138, U$175, U$212, U$249, U$286, U$323, U$64: (no value), buzzard_labels (11):R12
- added U$102, U$139, U$176, U$213, U$250, U$287, U$324, U$65: (no value), buzzard_labels (11):R23
- added U$103, U$140, U$177, U$214, U$251, U$288, U$325, U$66: (no value), buzzard_labels (11):VIN4
- added U$104, U$141, U$178, U$215, U$252, U$289, U$326, U$67: (no value), buzzard_labels (11):VMID5
- added U$105, U$142, U$179, U$216, U$253, U$290, U$327, U$68: (no value), buzzard_labels (11):VOUT6
- added U$106, U$107, U$143, U$144, U$180, U$181, U$217, U$218, U$254, U$255, U$291, U$292, U$328, U$329, U$69, U$70: (no value), buzzard_labels (12):CONFIGURABLE_RC_FILTER0
- added U$108, U$109, U$145, U$146, U$182, U$183, U$219, U$220, U$256, U$257, U$293, U$294, U$330, U$331, U$71, U$72: (no value), SparkFun-Hardware:STAND-OFF-TIGHT
- added U$110, U$147, U$184, U$221, U$258, U$295, U$332, U$73: (no value), SparkX:SPARKX-SMALL
- added U$111, U$148, U$185, U$222, U$259, U$296, U$333, U$74: (no value), SparkX:SPARKX-MEDIUM
- added U$112, U$149, U$186, U$223, U$260, U$297, U$38, U$75: (no value), buzzard_labels (6):1_#F9
- added U$113, U$150, U$187, U$224, U$261, U$298, U$39, U$76: (no value), buzzard_labels (6):1_KOHM7
- added U$114, U$151, U$188, U$225, U$262, U$299, U$40, U$77: (no value), buzzard_labels (6):10_#F8
- added U$115, U$152, U$189, U$226, U$263, U$300, U$41, U$78: (no value), buzzard_labels (6):10_MOHM6
- added U$116, U$117, U$153, U$154, U$190, U$191, U$227, U$228, U$264, U$265, U$301, U$302, U$42, U$43, U$79, U$80: (no value), buzzard_labels (7):GND0
- added U$118, U$119, U$155, U$156, U$192, U$193, U$229, U$230, U$266, U$267, U$303, U$304, U$44, U$45, U$81, U$82: (no value), buzzard_labels (7):VIN1
- added U$120, U$121, U$157, U$158, U$194, U$195, U$231, U$232, U$268, U$269, U$305, U$306, U$46, U$47, U$83, U$84: (no value), buzzard_labels (7):VMID3
- added U$122, U$123, U$159, U$160, U$196, U$197, U$233, U$234, U$270, U$271, U$307, U$308, U$48, U$49, U$85, U$86: (no value), buzzard_labels (8):VOUT3
- added U$124, U$161, U$198, U$235, U$272, U$309, U$50, U$87: (no value), buzzard_labels (6):10_NF11
- added U$125, U$162, U$199, U$236, U$273, U$310, U$51, U$88: (no value), buzzard_labels (6):10_OHM4
- added U$126, U$163, U$200, U$237, U$274, U$311, U$52, U$89: (no value), buzzard_labels (6):100_KOHM10
- added U$127, U$164, U$201, U$238, U$275, U$312, U$53, U$90: (no value), buzzard_labels (6):C10
- added U$128, U$165, U$202, U$239, U$276, U$313, U$54, U$91: (no value), buzzard_labels (6):C21
- added U$129, U$166, U$203, U$240, U$277, U$314, U$55, U$92: (no value), buzzard_labels (6):R12
- added U$130, U$167, U$204, U$241, U$278, U$315, U$56, U$93: (no value), buzzard_labels (6):R23
- added U$131, U$168, U$205, U$242, U$279, U$316, U$57, U$94: (no value), buzzard_labels (6):_1_OHM5
- added U$132, U$169, U$206, U$243, U$280, U$317, U$58, U$95: (no value), buzzard_labels (6):_1_PF13
- added U$133, U$170, U$207, U$244, U$281, U$318, U$59, U$96: (no value), buzzard_labels (6):_100_PF12
- added U$134, U$135, U$171, U$172, U$208, U$209, U$245, U$246, U$282, U$283, U$319, U$320, U$60, U$61, U$97, U$98: (no value), buzzard_labels (10):CUSTOM3
- added U$136, U$173, U$210, U$247, U$284, U$321, U$62, U$99: (no value), buzzard_labels (11):C11
Connections:
- new net GND1: C15.2, C16.2, C17.2, C18.2, C19.2, C20.-, C28.2, J2.1, R21.1, R22.1, R23.1, R24.1, R25.1, R26.P$1, R27.1
- new net GND2: C29.2, C30.2, C31.2, C32.2, C33.2, C34.-, C42.2, J3.1, R35.1, R36.1, R37.1, R38.1, R39.1, R40.P$1, R41.1
- new net GND3: C43.2, C44.2, C45.2, C46.2, C47.2, C48.-, C56.2, J4.1, R49.1, R50.1, R51.1, R52.1, R53.1, R54.P$1, R55.1
- new net GND4: C57.2, C58.2, C59.2, C60.2, C61.2, C62.-, C70.2, J5.1, R63.1, R64.1, R65.1, R66.1, R67.1, R68.P$1, R69.1
- new net GND5: C71.2, C72.2, C73.2, C74.2, C75.2, C76.-, C84.2, J6.1, R77.1, R78.1, R79.1, R80.1, R81.1, R82.P$1, R83.1
- new net GND6: C85.2, C86.2, C87.2, C88.2, C89.2, C90.-, C98.2, J7.1, R91.1, R92.1, R93.1, R94.1, R95.1, R96.P$1, R97.1
- new net GND7: C100.2, C101.2, C102.2, C103.2, C104.-, C112.2, C99.2, J8.1, R105.1, R106.1, R107.1, R108.1, R109.1, R110.P$1, R111.1
- new net GND8: C113.2, C114.2, C115.2, C116.2, C117.2, C118.-, C126.2, J9.1, R119.1, R120.1, R121.1, R122.1, R123.1, R124.P$1, R125.1
- new net N$100: R61.1, SW17.9
- new net N$101: R60.1, SW17.8
- new net N$102: R62.P$1, R70.1, SW17.7
- new net N$103: C57.1, SW18.7
- new net N$104: C58.1, SW18.8
- new net N$105: C59.1, SW18.9
- new net N$106: C60.1, SW18.10
- new net N$107: C61.1, SW18.11
- new net N$108: C62.+, C70.1, SW18.12
- new net N$109: R63.2, SW20.7
- new net N$110: R64.2, SW20.8
- new net N$111: R65.2, SW20.9
- new net N$112: R68.P$2, R69.2, SW20.12
- new net N$113: R66.2, SW20.11
- new net N$114: R67.2, SW20.10
- new net N$115: C68.+, C69.2, SW19.7
- new net N$116: C67.2, SW19.8
- new net N$117: C66.2, SW19.9
- new net N$118: C65.2, SW19.10
- new net N$119: C64.2, SW19.11
- new net N$120: C63.2, SW19.12
- new net N$121: R71.1, SW21.12
- new net N$122: R72.1, SW21.11
- new net N$123: R73.1, SW21.10
- new net N$124: R75.1, SW21.9
- new net N$125: R74.1, SW21.8
- new net N$126: R76.P$1, R84.1, SW21.7
- new net N$127: C71.1, SW22.7
- new net N$128: C72.1, SW22.8
- new net N$129: C73.1, SW22.9
- new net N$130: C74.1, SW22.10
- new net N$131: C75.1, SW22.11
- new net N$132: C76.+, C84.1, SW22.12
- new net N$133: R77.2, SW24.7
- new net N$134: R78.2, SW24.8
- new net N$135: R79.2, SW24.9
- new net N$136: R82.P$2, R83.2, SW24.12
- new net N$137: R80.2, SW24.11
- new net N$138: R81.2, SW24.10
- new net N$139: C82.+, C83.2, SW23.7
- new net N$140: C81.2, SW23.8
- new net N$141: C80.2, SW23.9
- new net N$142: C79.2, SW23.10
- new net N$143: C78.2, SW23.11
- new net N$144: C77.2, SW23.12
- new net N$145: R85.1, SW25.12
- new net N$146: R86.1, SW25.11
- new net N$147: R87.1, SW25.10
- new net N$148: R89.1, SW25.9
- new net N$149: R88.1, SW25.8
- new net N$150: R90.P$1, R98.1, SW25.7
- new net N$151: C85.1, SW26.7
- new net N$152: C86.1, SW26.8
- new net N$153: C87.1, SW26.9
- new net N$154: C88.1, SW26.10
- new net N$155: C89.1, SW26.11
- new net N$156: C90.+, C98.1, SW26.12
- new net N$157: R91.2, SW28.7
- new net N$158: R92.2, SW28.8
- new net N$159: R93.2, SW28.9
- new net N$160: R96.P$2, R97.2, SW28.12
- new net N$161: R94.2, SW28.11
- new net N$162: R95.2, SW28.10
- new net N$163: C96.+, C97.2, SW27.7
- new net N$164: C95.2, SW27.8
- new net N$165: C94.2, SW27.9
- new net N$166: C93.2, SW27.10
- new net N$167: C92.2, SW27.11
- new net N$168: C91.2, SW27.12
- new net N$169: R99.1, SW29.12
- new net N$170: R100.1, SW29.11
- new net N$171: R101.1, SW29.10
- new net N$172: R103.1, SW29.9
- new net N$173: R102.1, SW29.8
- new net N$174: R104.P$1, R112.1, SW29.7
- new net N$175: C99.1, SW30.7
- new net N$176: C100.1, SW30.8
- new net N$177: C101.1, SW30.9
- new net N$178: C102.1, SW30.10
- new net N$179: C103.1, SW30.11
- new net N$180: C104.+, C112.1, SW30.12
- new net N$181: R105.2, SW32.7
- new net N$182: R106.2, SW32.8
- new net N$183: R107.2, SW32.9
- new net N$184: R110.P$2, R111.2, SW32.12
- new net N$185: R108.2, SW32.11
- new net N$186: R109.2, SW32.10
- new net N$187: C110.+, C111.2, SW31.7
- new net N$188: C109.2, SW31.8
- new net N$189: C108.2, SW31.9
- new net N$190: C107.2, SW31.10
- new net N$191: C106.2, SW31.11
- new net N$192: C105.2, SW31.12
- new net N$193: R113.1, SW33.12
- new net N$194: R114.1, SW33.11
- new net N$195: R115.1, SW33.10
- new net N$196: R117.1, SW33.9
- new net N$197: R116.1, SW33.8
- new net N$198: R118.P$1, R126.1, SW33.7
- new net N$199: C113.1, SW34.7
- new net N$200: C114.1, SW34.8
- new net N$201: C115.1, SW34.9
- new net N$202: C116.1, SW34.10
- new net N$203: C117.1, SW34.11
- new net N$204: C118.+, C126.1, SW34.12
- new net N$205: R119.2, SW36.7
- new net N$206: R120.2, SW36.8
- new net N$207: R121.2, SW36.9
- new net N$208: R124.P$2, R125.2, SW36.12
- new net N$209: R122.2, SW36.11
- new net N$210: R123.2, SW36.10
- new net N$211: C124.+, C125.2, SW35.7
- new net N$212: C123.2, SW35.8
- new net N$213: C122.2, SW35.9
- new net N$214: C121.2, SW35.10
- new net N$215: C120.2, SW35.11
- new net N$216: C119.2, SW35.12
- new net N$25: R15.1, SW5.12
- new net N$26: R16.1, SW5.11
- new net N$27: R17.1, SW5.10
- new net N$28: R19.1, SW5.9
- new net N$29: R18.1, SW5.8
- new net N$30: R20.P$1, R28.1, SW5.7
- new net N$31: C15.1, SW6.7
- new net N$32: C16.1, SW6.8
- new net N$33: C17.1, SW6.9
- new net N$34: C18.1, SW6.10
- new net N$35: C19.1, SW6.11
- new net N$36: C20.+, C28.1, SW6.12
- new net N$37: R21.2, SW8.7
- new net N$38: R22.2, SW8.8
- new net N$39: R23.2, SW8.9
- new net N$40: R26.P$2, R27.2, SW8.12
- new net N$41: R24.2, SW8.11
- new net N$42: R25.2, SW8.10
- new net N$43: C26.+, C27.2, SW7.7
- new net N$44: C25.2, SW7.8
- new net N$45: C24.2, SW7.9
- new net N$46: C23.2, SW7.10
- new net N$47: C22.2, SW7.11
- new net N$48: C21.2, SW7.12
- new net N$49: R29.1, SW9.12
- new net N$50: R30.1, SW9.11
- new net N$51: R31.1, SW9.10
- new net N$52: R33.1, SW9.9
- new net N$53: R32.1, SW9.8
- new net N$54: R34.P$1, R42.1, SW9.7
- new net N$55: C29.1, SW10.7
- new net N$56: C30.1, SW10.8
- new net N$57: C31.1, SW10.9
- new net N$58: C32.1, SW10.10
- new net N$59: C33.1, SW10.11
- new net N$60: C34.+, C42.1, SW10.12
- new net N$61: R35.2, SW12.7
- new net N$62: R36.2, SW12.8
- new net N$63: R37.2, SW12.9
- new net N$64: R40.P$2, R41.2, SW12.12
- new net N$65: R38.2, SW12.11
- new net N$66: R39.2, SW12.10
- new net N$67: C40.+, C41.2, SW11.7
- new net N$68: C39.2, SW11.8
- new net N$69: C38.2, SW11.9
- new net N$70: C37.2, SW11.10
- new net N$71: C36.2, SW11.11
- new net N$72: C35.2, SW11.12
- new net N$73: R43.1, SW13.12
- new net N$74: R44.1, SW13.11
- new net N$75: R45.1, SW13.10
- new net N$76: R47.1, SW13.9
- new net N$77: R46.1, SW13.8
- new net N$78: R48.P$1, R56.1, SW13.7
- new net N$79: C43.1, SW14.7
- new net N$80: C44.1, SW14.8
- new net N$81: C45.1, SW14.9
- new net N$82: C46.1, SW14.10
- new net N$83: C47.1, SW14.11
- new net N$84: C48.+, C56.1, SW14.12
- new net N$85: R49.2, SW16.7
- new net N$86: R50.2, SW16.8
- new net N$87: R51.2, SW16.9
- new net N$88: R54.P$2, R55.2, SW16.12
- new net N$89: R52.2, SW16.11
- new net N$90: R53.2, SW16.10
- new net N$91: C54.+, C55.2, SW15.7
- new net N$92: C53.2, SW15.8
- new net N$93: C52.2, SW15.9
- new net N$94: C51.2, SW15.10
- new net N$95: C50.2, SW15.11
- new net N$96: C49.2, SW15.12
- new net N$97: R57.1, SW17.12
- new net N$98: R58.1, SW17.11
- new net N$99: R59.1, SW17.10
- new net VDDA1: J2.3, R15.2, R16.2, R17.2, R18.2, R19.2, R20.P$2, R28.2, SW6.1, SW6.2, SW6.3, SW6.4, SW6.5, SW6.6, SW7.1, SW7.2, SW7.3, SW7.4, SW7.5, SW7.6
- new net VDDA2: J3.3, R29.2, R30.2, R31.2, R32.2, R33.2, R34.P$2, R42.2, SW10.1, SW10.2, SW10.3, SW10.4, SW10.5, SW10.6, SW11.1, SW11.2, SW11.3, SW11.4, SW11.5, SW11.6
- new net VDDA3: J4.3, R43.2, R44.2, R45.2, R46.2, R47.2, R48.P$2, R56.2, SW14.1, SW14.2, SW14.3, SW14.4, SW14.5, SW14.6, SW15.1, SW15.2, SW15.3, SW15.4, SW15.5, SW15.6
- new net VDDA4: J5.3, R57.2, R58.2, R59.2, R60.2, R61.2, R62.P$2, R70.2, SW18.1, SW18.2, SW18.3, SW18.4, SW18.5, SW18.6, SW19.1, SW19.2, SW19.3, SW19.4, SW19.5, SW19.6
- new net VDDA5: J6.3, R71.2, R72.2, R73.2, R74.2, R75.2, R76.P$2, R84.2, SW22.1, SW22.2, SW22.3, SW22.4, SW22.5, SW22.6, SW23.1, SW23.2, SW23.3, SW23.4, SW23.5, SW23.6
- new net VDDA6: J7.3, R85.2, R86.2, R87.2, R88.2, R89.2, R90.P$2, R98.2, SW26.1, SW26.2, SW26.3, SW26.4, SW26.5, SW26.6, SW27.1, SW27.2, SW27.3, SW27.4, SW27.5, SW27.6
- new net VDDA7: J8.3, R100.2, R101.2, R102.2, R103.2, R104.P$2, R112.2, R99.2, SW30.1, SW30.2, SW30.3, SW30.4, SW30.5, SW30.6, SW31.1, SW31.2, SW31.3, SW31.4, SW31.5, SW31.6
- new net VDDA8: J9.3, R113.2, R114.2, R115.2, R116.2, R117.2, R118.P$2, R126.2, SW34.1, SW34.2, SW34.3, SW34.4, SW34.5, SW34.6, SW35.1, SW35.2, SW35.3, SW35.4, SW35.5, SW35.6
- new net VIN1: J2.4, SW5.1, SW5.2, SW5.3, SW5.4, SW5.5, SW5.6
- new net VIN2: J3.4, SW9.1, SW9.2, SW9.3, SW9.4, SW9.5, SW9.6
- new net VIN3: J4.4, SW13.1, SW13.2, SW13.3, SW13.4, SW13.5, SW13.6
- new net VIN4: J5.4, SW17.1, SW17.2, SW17.3, SW17.4, SW17.5, SW17.6
- new net VIN5: J6.4, SW21.1, SW21.2, SW21.3, SW21.4, SW21.5, SW21.6
- new net VIN6: J7.4, SW25.1, SW25.2, SW25.3, SW25.4, SW25.5, SW25.6
- new net VIN7: J8.4, SW29.1, SW29.2, SW29.3, SW29.4, SW29.5, SW29.6
- new net VIN8: J9.4, SW33.1, SW33.2, SW33.3, SW33.4, SW33.5, SW33.6
- new net VOUT1: C21.1, C22.1, C23.1, C24.1, C25.1, C26.-, C27.1, J2.2, SW8.1, SW8.2, SW8.3, SW8.4, SW8.5, SW8.6
- new net VOUT2: C35.1, C36.1, C37.1, C38.1, C39.1, C40.-, C41.1, J3.2, SW12.1, SW12.2, SW12.3, SW12.4, SW12.5, SW12.6
- new net VOUT3: C49.1, C50.1, C51.1, C52.1, C53.1, C54.-, C55.1, J4.2, SW16.1, SW16.2, SW16.3, SW16.4, SW16.5, SW16.6
- new net VOUT4: C63.1, C64.1, C65.1, C66.1, C67.1, C68.-, C69.1, J5.2, SW20.1, SW20.2, SW20.3, SW20.4, SW20.5, SW20.6
- new net VOUT5: C77.1, C78.1, C79.1, C80.1, C81.1, C82.-, C83.1, J6.2, SW24.1, SW24.2, SW24.3, SW24.4, SW24.5, SW24.6
- new net VOUT6: C91.1, C92.1, C93.1, C94.1, C95.1, C96.-, C97.1, J7.2, SW28.1, SW28.2, SW28.3, SW28.4, SW28.5, SW28.6
- new net VOUT7: C105.1, C106.1, C107.1, C108.1, C109.1, C110.-, C111.1, J8.2, SW32.1, SW32.2, SW32.3, SW32.4, SW32.5, SW32.6
- new net VOUT8: C119.1, C120.1, C121.1, C122.1, C123.1, C124.-, C125.1, J9.2, SW36.1, SW36.2, SW36.3, SW36.4, SW36.5, SW36.6
Routing:
- net VDDA7: track 0.00 -> 144.8 mm
- net VDDA4: track 0.00 -> 144.8 mm
- net VDDA1: track 0.00 -> 144.8 mm
- net VDDA5: track 0.00 -> 144.8 mm
- net VDDA3: track 0.00 -> 144.8 mm
- net VDDA2: track 0.00 -> 144.8 mm
- net VDDA8: track 0.00 -> 144.8 mm
- net VDDA6: track 0.00 -> 144.8 mm
- net VOUT1: track 0.00 -> 89.3 mm
- net VOUT7: track 0.00 -> 89.3 mm
- net VOUT4: track 0.00 -> 89.3 mm
- net VOUT6: track 0.00 -> 89.3 mm
- net VOUT3: track 0.00 -> 89.3 mm
- net VOUT2: track 0.00 -> 89.3 mm
- net VOUT5: track 0.00 -> 89.3 mm
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- added copper zone on layer 1, net GND1
- added copper zone on layer 16, net GND1
- added copper zone on layer 1, net GND2
- added copper zone on layer 16, net GND2
- added copper zone on layer 1, net GND3
- added copper zone on layer 16, net GND3
- added copper zone on layer 1, net GND4
- added copper zone on layer 16, net GND4
- added copper zone on layer 1, net GND5
- added copper zone on layer 16, net GND5
- added copper zone on layer 1, net GND6
- added copper zone on layer 16, net GND6
- added copper zone on layer 1, net GND7
- added copper zone on layer 16, net GND7
- added copper zone on layer 1, net GND8
- added copper zone on layer 16, net GND8
Other:
- board size 48.3 x 40.6 mm -> 165.9 x 143 mm
- board text added: "v-score"
- board text removed: "Andy England"
